File: limit_switch_board/switch_board.kicad_pcb (KiCad board)
At the start: 2 copper layers, 38.4 x 28.4 mm, 9 parts, among them J1 CONN_01X04, J2 CONN_01X03

Commit message: minor board fixes: limit switches and stepper motors
Other:
- board text added: "+"
Changed lines of the file:
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@@
-(kicad_pcb (version 4) (host pcbnew 4.0.7-e0-6372~58~ubuntu16.04.1)
+(kicad_pcb (version 4) (host pcbnew 4.0.7-e2-6376~58~ubuntu16.04.1)
   (general
     (links 11)
@@
     (area 126.6092 32.055999 165.302001 60.7338)
     (thickness 1.6)
-    (drawings 4)
+    (drawings 5)
     (tracks 37)
     (zones 0)
@@
     (pad 1 np_thru_hole circle (at 0 0) (size 3.2 3.2) (drill 3.2) (layers *.Cu *.Mask))
   )
+  (gr_text + (at 136 46.5) (layer F.SilkS)
+    (effects (font (size 1.5 1.5) (thickness 0.3)))
+  )
   (gr_line (start 165.227 60.5409) (end 165.227 32.131) (angle 90) (layer Edge.Cuts) (width 0.15))
