File: stepper_drivers_board/stepper_drivers.kicad_pcb (KiCad board)
At the start: 2 copper layers, 41.5 x 76.5 mm, 29 parts

Commit message: Fix a typo in the steppers board
Parts:
- LIMZ Y X: renamed from LIMZ X Y
Changed lines of the file:
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@@
     (descr "Through hole straight pin header, 1x03, 2.54mm pitch, single row")
     (tags "Through hole pin header THT 1x03 2.54mm single row")
-    (fp_text reference "LIMZ X Y" (at -2.5 3.5 90) (layer F.SilkS)
+    (fp_text reference "LIMZ Y X" (at -2.5 3.5 90) (layer F.SilkS)
       (effects (font (size 1 1) (thickness 0.15)))
     )
