File: stepper_with_uc_board/stepper_drivers.sch (KiCad schematic (older format))
At the start: 36 parts, among them J1 Conn_02x03_Odd_Even, U1 LM317_3PinPackage, U2 ATMEGA328P-AU, Y1 16MHz

Commit message: Additional text and some footprint fixes
Parts:
- U2: footprint Housings_QFP:TQFP-32_7x7mm_Pitch0.8mm -> My Shit:My_TQFP-32_7x7mm_Pitch0.8mm
Changed lines of the file:
@@
 F 0 "U2" H 1600 5900 50  0000 L BNN
 F 1 "ATMEGA328P-AU" H 2750 3250 50  0000 L BNN
-F 2 "Housings_QFP:TQFP-32_7x7mm_Pitch0.8mm" H 2350 4650 50  0001 C CIN
+F 2 "My Shit:My_TQFP-32_7x7mm_Pitch0.8mm" H 2350 4650 50  0001 C CIN
 F 3 "" H 2350 4650 50  0001 C CNN
 	1    2350 4650
