File: stepper_with_uc_board/stepper_drivers.kicad_pcb (KiCad board)
At the start: 2 copper layers, 56.2 x 76.5 mm, 40 parts, among them U1 LM317_3PinPackage, U2 ATMEGA328P-AU, Y1 16MHz

Commit message: Additional text and some footprint fixes
Parts:
- LIM:Z   Y   X: renamed from LIM: Z    Y     X
- U2: footprint Housings_QFP:TQFP-32_7x7mm_Pitch0.8mm -> My Shit:My_TQFP-32_7x7mm_Pitch0.8mm
Connections:
- U2 pad 18: (no net) -> Net-(U2-Pad18)
- U2 pad 19: (no net) -> Net-(U2-Pad19)
- U2 pad 20: (no net) -> Net-(U2-Pad20)
- U2 pad 22: (no net) -> Net-(U2-Pad22)
- U2 pad 23: (no net) -> Net-(U2-Pad23)
- U2 pad 24: (no net) -> Net-(U2-Pad24)
- U2 pad 25: (no net) -> Net-(U2-Pad25)
- U2 pad 26: (no net) -> Net-(U2-Pad26)
- U2 pad 27: (no net) -> Net-(U2-Pad27)
- U2 pad 28: (no net) -> Net-(U2-Pad28)
Other:
- net class Chubby: clearance 0.25 -> 0.45
- board text added: "12V"
- board text added: "GND"
- board text added: "SIG"
- board text added: "https://github.com/jonronen/kicad-stuff"

Commit message: more minor fixes to the UC with stepper drivers board
Routing:
- net Net-(U2-Pad1): track 23.4 -> 25.4 mm
- net Net-(J1-Pad5): track 52.5 -> 51.3 mm
Other:
- board text added: "C3E5"
- board text added: "https://github.com/c3e5/lazer"
- board text removed: "https://github.com/jonronen/kicad-stuff"
